Commit message: try

File: src/SimpleArm/urdf/SimpleArm.xacro (robot description, xacro)
@@ -1,7 +1,8 @@
-<robot name="SimpleArm">
+<?xml version="1.0"?>
+<robot name="SimpleArm"  xmlns:xacro="http://www.ros.org/wiki/xacro">
   <xacro:property name="altura_base" value="0.1"/>
   <xacro:property name="largo" value="0.5"/>
   <xacro:property name="ancho" value="0.1"/>
-  <xacro:property name="masa" value="2"/>
+  <xacro:property name="masa" value="2.0"/>
   <link name="link0">
     <visual>
@@ -17,5 +18,5 @@
       <origin xyz="0 0 0" rpy="0 0 0" />
     </colission>
-    <xacro:default_inertial_mass="1000"/>
+    <xacro:default_inertial mass="1000"/>
   </link>
   <link name="link1">
@@ -32,5 +33,5 @@
       <origin xyz="0 0 0" rpy="0 0 0" />
     </colission>
-    <xacro:default_inertial_mass="${masa}"/>
+    <xacro:default_inertial mass="${masa}"/>
   </link>
   <link name="link2">
@@ -47,5 +48,5 @@
       <origin xyz="0 0 0" rpy="0 0 0" />
     </colission>
-    <xacro:default_inertial_mass="${masa}"/>
+    <xacro:default_inertial mass="${masa}"/>
   </link>
   <link name="link3">
@@ -62,5 +63,5 @@
       <origin xyz="0 0 0" rpy="0 0 0" />
     </colission>
-    <xacro:default_inertial_mass="${masa}"/>
+    <xacro:default_inertial mass="${masa}"/>
   </link>
   <link name="link4">
@@ -77,5 +78,5 @@
       <origin xyz="0 0 0" rpy="0 0 0" />
     </colission>
-    <xacro:default_inertial_mass="${masa}"/>
+    <xacro:default_inertial mass="${masa}"/>
   </link>
   <joint name="joint1" type="continuous">

Commit message: Fixed xacro

File: src/SimpleArm/urdf/SimpleArm.xacro (robot description, xacro)
@@ -5,4 +5,10 @@
   <xacro:property name="ancho" value="0.1"/>
   <xacro:property name="masa" value="2.0"/>
+<xacro:macro name="default_inertial" params="mass">
+	<inertial>
+		<mass value="${mass}"/>
+		<inertia ixx="1.0" ixy="0.0" ixz="0.0" iyy="1.0" iyz="0.0" izz="1.0"/>
+	</inertial>
+</xacro:macro>
   <link name="link0">
     <visual>

Commit message: Fixed urdf collision tag and joint placement
Fixed typo in collision tag of all links and corrected joint origins

File: src/SimpleArm/urdf/SimpleArm.xacro (robot description, xacro)
@@ -5,24 +5,25 @@
   <xacro:property name="ancho" value="0.1"/>
   <xacro:property name="masa" value="2.0"/>
-<xacro:macro name="default_inertial" params="mass">
-	<inertial>
-		<mass value="${mass}"/>
-		<inertia ixx="1.0" ixy="0.0" ixz="0.0" iyy="1.0" iyz="0.0" izz="1.0"/>
-	</inertial>
+<xacro:macro name="default_inertial" params="mass altoL">
+  <inertial>
+    <origin xyz="0 0 ${altoL/2}" rpy="0 0 0"/>
+    <mass value="${mass}"/>
+    <inertia ixx="1.0" ixy="0.0" ixz="0.0" iyy="1.0" iyz="0.0" izz="1.0"/>
+  </inertial>
 </xacro:macro>
   <link name="link0">
     <visual>
+      <origin xyz="0 0 ${altura_base/2}" rpy="0 0 0"/>
       <geometry>
         <box size="1 1 ${altura_base}"/>
       </geometry>
-      <origin xyz="0 0 0" rpy="0 0 0" />
     </visual>
-    <colission>
+    <collision>
+      <origin xyz="0 0 ${altura_base/2}" rpy="0 0 0"/>
       <geometry>
         <box size="1 1 ${altura_base}"/>
       </geometry>
-      <origin xyz="0 0 0" rpy="0 0 0" />
-    </colission>
-    <xacro:default_inertial mass="1000"/>
+    </collision>
+   <xacro:default_inertial mass="1000" altoL="${altura_base}"/>
   </link>
   <link name="link1">
@@ -31,13 +32,13 @@
         <cylinder radius="${ancho}" length="${largo}"/>
       </geometry>
-      <origin xyz="0 0 0" rpy="0 0 0" />
+      <origin xyz="0 0 ${largo/2}" rpy="0 0 0" />
     </visual>
-    <colission>
+    <collission>
       <geometry>
          <cylinder radius="${ancho}" length="${largo}"/>
       </geometry>
-      <origin xyz="0 0 0" rpy="0 0 0" />
-    </colission>
-    <xacro:default_inertial mass="${masa}"/>
+      <origin xyz="0 0 ${largo/2}" rpy="0 0 0" />
+    </collission>
+    <xacro:default_inertial mass="${masa}" altoL="${largo}"/>
   </link>
   <link name="link2">
@@ -46,5 +47,5 @@
         <cylinder radius="${ancho}" length="${largo}"/>
       </geometry>
-      <origin xyz="0 0 0" rpy="0 0 0" />
+      <origin xyz="0 0 ${largo/2}" rpy="0 0 0" />
     </visual>
     <colission>
@@ -52,7 +53,7 @@
          <cylinder radius="${ancho}" length="${largo}"/>
       </geometry>
-      <origin xyz="0 0 0" rpy="0 0 0" />
+      <origin xyz="0 0 ${largo/2}" rpy="0 0 0" />
     </colission>
-    <xacro:default_inertial mass="${masa}"/>
+    <xacro:default_inertial mass="${masa}" altoL="${largo}"/>
   </link>
   <link name="link3">
@@ -61,5 +62,5 @@
         <cylinder radius="${ancho}" length="${largo}"/>
       </geometry>
-      <origin xyz="0 0 0" rpy="0 0 0" />
+      <origin xyz="0 0 ${largo/2}" rpy="0 0 0" />
     </visual>
     <colission>
@@ -67,7 +68,7 @@
          <cylinder radius="${ancho}" length="${largo}"/>
       </geometry>
-      <origin xyz="0 0 0" rpy="0 0 0" />
+      <origin xyz="0 0 ${largo/2}" rpy="0 0 0" />
     </colission>
-    <xacro:default_inertial mass="${masa}"/>
+    <xacro:default_inertial mass="${masa}" altoL="${largo}"/>
   </link>
   <link name="link4">
@@ -76,5 +77,5 @@
         <cylinder radius="${ancho}" length="${largo}"/>
       </geometry>
-      <origin xyz="0 0 0" rpy="0 0 0" />
+      <origin xyz="0 0 ${largo/2}" rpy="0 0 0" />
     </visual>
     <colission>
@@ -82,7 +83,7 @@
          <cylinder radius="${ancho}" length="${largo}"/>
       </geometry>
-      <origin xyz="0 0 0" rpy="0 0 0" />
+      <origin xyz="0 0 ${largo/2}" rpy="0 0 0" />
     </colission>
-    <xacro:default_inertial mass="${masa}"/>
+    <xacro:default_inertial mass="${masa}" altoL="${largo}"/>
   </link>
   <joint name="joint1" type="continuous">
@@ -90,19 +91,23 @@
     <child link="link1"/>
     <origin xyz="0 0 ${altura_base}" rpy="0 0 0" />
+    <axis xyz="0 0 1"/>
   </joint>
   <joint name="joint2" type="continuous">
     <parent link="link1"/>
     <child link="link2"/>
-    <origin xyz="0 0 ${largo+altura_base}" rpy="0 0 0" />
+    <origin xyz="0 0 ${largo}" rpy="0 0 0" />
+    <axis xyz="0 1 0"/>
   </joint>
   <joint name="joint3" type="continuous">
     <parent link="link2"/>
     <child link="link3"/>
-    <origin xyz="0 0 ${largo*2+altura_base}" rpy="0 0 0" />
+    <origin xyz="0 0 ${largo}" rpy="0 0 0" />
+    <axis xyz="0 1 0"/>
   </joint>
   <joint name="joint4" type="continuous">
     <parent link="link3"/>
     <child link="link4"/>
-    <origin xyz="0 0 ${largo*3+altura_base}" rpy="0 0 0" />
+    <origin xyz="0 0 ${largo}" rpy="0 0 0" />
+    <axis xyz="0 1 0"/>
   </joint>
 </robot>

Commit message: Added joint dynamic damping

File: src/SimpleArm/urdf/SimpleArm.xacro (robot description, xacro)
@@ -92,4 +92,5 @@
     <origin xyz="0 0 ${altura_base}" rpy="0 0 0" />
     <axis xyz="0 0 1"/>
+    <dynamics damping="0.6"/>
   </joint>
   <joint name="joint2" type="continuous">
@@ -98,4 +99,5 @@
     <origin xyz="0 0 ${largo}" rpy="0 0 0" />
     <axis xyz="0 1 0"/>
+    <dynamics damping="0.6"/>
   </joint>
   <joint name="joint3" type="continuous">
@@ -104,4 +106,5 @@
     <origin xyz="0 0 ${largo}" rpy="0 0 0" />
     <axis xyz="0 1 0"/>
+    <dynamics damping="0.6"/>
   </joint>
   <joint name="joint4" type="continuous">
@@ -110,4 +113,5 @@
     <origin xyz="0 0 ${largo}" rpy="0 0 0" />
     <axis xyz="0 1 0"/>
+    <dynamics damping="0.6"/>
   </joint>
 </robot>

Commit message: Added self collision and colors for links, fixed collision tag

File: src/SimpleArm/urdf/SimpleArm.xacro (robot description, xacro)
@@ -5,11 +5,14 @@
   <xacro:property name="ancho" value="0.1"/>
   <xacro:property name="masa" value="2.0"/>
-<xacro:macro name="default_inertial" params="mass altoL">
-  <inertial>
-    <origin xyz="0 0 ${altoL/2}" rpy="0 0 0"/>
-    <mass value="${mass}"/>
-    <inertia ixx="1.0" ixy="0.0" ixz="0.0" iyy="1.0" iyz="0.0" izz="1.0"/>
-  </inertial>
-</xacro:macro>
+  <xacro:macro name="default_inertial" params="mass altoL">
+    <inertial>
+      <origin xyz="0 0 ${altoL/2}" rpy="0 0 0"/>
+      <mass value="${mass}"/>
+      <inertia ixx="1.0" ixy="0.0" ixz="0.0" iyy="1.0" iyz="0.0" izz="1.0"/>
+    </inertial>
+  </xacro:macro>
+  <xacro:include filename="$(find SimpleArm)/urdf/SimpleArm.gazebo" />
+   <!-- Import Rviz colors -->
+<xacro:include filename="$(find SimpleArm)/urdf/materials.xacro" />
   <link name="link0">
     <visual>
@@ -33,11 +36,12 @@
       </geometry>
       <origin xyz="0 0 ${largo/2}" rpy="0 0 0" />
+      <material name="orange"/>
     </visual>
-    <collission>
+    <collision>
       <geometry>
          <cylinder radius="${ancho}" length="${largo}"/>
       </geometry>
       <origin xyz="0 0 ${largo/2}" rpy="0 0 0" />
-    </collission>
+    </collision>
     <xacro:default_inertial mass="${masa}" altoL="${largo}"/>
   </link>
@@ -48,11 +52,12 @@
       </geometry>
       <origin xyz="0 0 ${largo/2}" rpy="0 0 0" />
+      <material name="white"/>
     </visual>
-    <colission>
+    <collision>
       <geometry>
          <cylinder radius="${ancho}" length="${largo}"/>
       </geometry>
       <origin xyz="0 0 ${largo/2}" rpy="0 0 0" />
-    </colission>
+    </collision>
     <xacro:default_inertial mass="${masa}" altoL="${largo}"/>
   </link>
@@ -63,11 +68,12 @@
       </geometry>
       <origin xyz="0 0 ${largo/2}" rpy="0 0 0" />
+      <material name="orange"/>
     </visual>
-    <colission>
+    <collision>
       <geometry>
          <cylinder radius="${ancho}" length="${largo}"/>
       </geometry>
       <origin xyz="0 0 ${largo/2}" rpy="0 0 0" />
-    </colission>
+    </collision>
     <xacro:default_inertial mass="${masa}" altoL="${largo}"/>
   </link>
@@ -78,11 +84,12 @@
       </geometry>
       <origin xyz="0 0 ${largo/2}" rpy="0 0 0" />
+      <material name="white"/>
     </visual>
-    <colission>
+    <collision>
       <geometry>
          <cylinder radius="${ancho}" length="${largo}"/>
       </geometry>
       <origin xyz="0 0 ${largo/2}" rpy="0 0 0" />
-    </colission>
+    </collision>
     <xacro:default_inertial mass="${masa}" altoL="${largo}"/>
   </link>

Commit message: Adds ros controllers

File: src/SimpleArm/urdf/SimpleArm.xacro (robot description, xacro)
@@ -122,3 +122,44 @@
     <dynamics damping="0.6"/>
   </joint>
+  <!-- Transmission -->
+  <transmission name="tran1">
+    <type>transmission_interface/SimpleTransmission</type>
+    <joint name="joint1">
+      <hardwareInterface>hardware_interface/EffortJointInterface</hardwareInterface>
+    </joint>
+    <actuator name="yaw">
+      <hardwareInterface>hardware_interface/EffortJointInterface</hardwareInterface>
+      <mechanicalReduction>1</mechanicalReduction>
+    </actuator>
+  </transmission>
+  <transmission name="tran2">
+    <type>transmission_interface/SimpleTransmission</type>
+    <joint name="joint2">
+      <hardwareInterface>hardware_interface/EffortJointInterface</hardwareInterface>
+    </joint>
+    <actuator name="pitch1">
+      <hardwareInterface>hardware_interface/EffortJointInterface</hardwareInterface>
+      <mechanicalReduction>1</mechanicalReduction>
+    </actuator>
+</transmission>
+<transmission name="tran3">
+    <type>transmission_interface/SimpleTransmission</type>
+    <joint name="joint3">
+      <hardwareInterface>hardware_interface/EffortJointInterface</hardwareInterface>
+    </joint>
+    <actuator name="pitch2">
+      <hardwareInterface>hardware_interface/EffortJointInterface</hardwareInterface>
+      <mechanicalReduction>1</mechanicalReduction>
+    </actuator>
+  </transmission>
+  <transmission name="tran4">
+    <type>transmission_interface/SimpleTransmission</type>
+    <joint name="joint4">
+      <hardwareInterface>hardware_interface/EffortJointInterface</hardwareInterface>
+    </joint>
+    <actuator name="pitch3">
+      <hardwareInterface>hardware_interface/EffortJointInterface</hardwareInterface>
+      <mechanicalReduction>1</mechanicalReduction>
+    </actuator>
+</transmission>
 </robot>

Commit message: adjust pid and add sphere to the end of the arm

File: src/SimpleArm/urdf/SimpleArm.xacro (robot description, xacro)
@@ -1,8 +1,10 @@
 <?xml version="1.0"?>
 <robot name="SimpleArm"  xmlns:xacro="http://www.ros.org/wiki/xacro">
+  <link name="world"/>
   <xacro:property name="altura_base" value="0.1"/>
   <xacro:property name="largo" value="0.5"/>
   <xacro:property name="ancho" value="0.1"/>
-  <xacro:property name="masa" value="2.0"/>
+  <xacro:property name="masa" value="5"/>
+  <xacro:property name="delta" value="0.1"/>
   <xacro:macro name="default_inertial" params="mass altoL">
     <inertial>
@@ -28,5 +30,5 @@
       </geometry>
     </collision>
-   <xacro:default_inertial mass="1000000" altoL="${altura_base}"/>
+   <xacro:default_inertial mass="1000" altoL="${altura_base}"/>
   </link>
   <link name="link1">
@@ -94,4 +96,24 @@
     <xacro:default_inertial mass="${masa}" altoL="${largo}"/>
   </link>
+  <link name="link5">
+    <visual>
+      <geometry>
+        <sphere radius="${ancho}"/>
+      </geometry>
+      <origin xyz="0 0 ${ancho}" rpy="0 0 0" />
+      <material name="orange"/>
+    </visual>
+    <collision>
+      <geometry>
+        <sphere radius="${ancho}"/>
+      </geometry>
+      <origin xyz="0 0 ${ancho}" rpy="0 0 0" />
+    </collision>
+    <xacro:default_inertial mass="${masa/20}" altoL="${ancho}"/>
+  </link>
+  <joint name="joint0" type="fixed">
+    <parent link="world"/>
+    <child link="link0"/>
+  </joint>
   <joint name="joint1" type="continuous">
     <parent link="link0"/>
@@ -104,5 +126,5 @@
     <parent link="link1"/>
     <child link="link2"/>
-    <origin xyz="0 0 ${largo}" rpy="0 0 0" />
+    <origin xyz="0 0 ${largo+delta}" rpy="0 0 0" />
     <axis xyz="0 1 0"/>
     <dynamics damping="0.6"/>
@@ -111,5 +133,5 @@
     <parent link="link2"/>
     <child link="link3"/>
-    <origin xyz="0 0 ${largo}" rpy="0 0 0" />
+    <origin xyz="0 0 ${largo+delta}" rpy="0 0 0" />
     <axis xyz="0 1 0"/>
     <dynamics damping="0.6"/>
@@ -118,8 +140,13 @@
     <parent link="link3"/>
     <child link="link4"/>
-    <origin xyz="0 0 ${largo}" rpy="0 0 0" />
+    <origin xyz="0 0 ${largo+delta}" rpy="0 0 0" />
     <axis xyz="0 1 0"/>
     <dynamics damping="0.6"/>
   </joint>
+  <joint name="joint5" type="fixed">
+    <parent link="link4"/>
+    <child link="link5"/>
+    <origin xyz="0 0 ${largo}" rpy="0 0 0" />
+    </joint>
   <!-- Transmission -->
   <transmission name="tran1">

Commit message: fix inercia

File: src/SimpleArm/urdf/SimpleArm.xacro (robot description, xacro)
@@ -7,9 +7,23 @@
   <xacro:property name="masa" value="5"/>
   <xacro:property name="delta" value="0.1"/>
-  <xacro:macro name="default_inertial" params="mass altoL">
+  <xacro:macro name="cuboid_inertia_def" params="x y z mass">
     <inertial>
-      <origin xyz="0 0 ${altoL/2}" rpy="0 0 0"/>
+      <origin xyz="0 0 ${z/2}" rpy="0 0 0"/>
       <mass value="${mass}"/>
-      <inertia ixx="1.0" ixy="0.0" ixz="0.0" iyy="1.0" iyz="0.0" izz="1.0"/>
+      <inertia
+        iyy="${mass*(z*z+x*x)/12.0}"
+        ixx="${mass*(y*y+z*z)/12.0}"
+        izz="${mass*(x*x+y*y)/12.0}"
+        ixy="0.0" iyz="0.0" ixz="0.0"/>
+    </inertial>
+  </xacro:macro>
+  <xacro:macro name="default_inertial" params="mass length radius">
+    <inertial>
+      <origin xyz="0 0 ${length/2}" rpy="0 0 0"/>
+      <mass value="${mass}"/>
+          <inertia ixx="${mass*(3.0*radius*radius+length*length)/12.0}"
+             iyy="${mass*(3.0*radius*radius+length*length)/12.0}"
+             izz="${mass*radius*radius/2.0}"
+             ixy="0.0" iyz="0.0" ixz="0.0"/>
     </inertial>
   </xacro:macro>
@@ -30,5 +44,5 @@
       </geometry>
     </collision>
-   <xacro:default_inertial mass="1000" altoL="${altura_base}"/>
+   <xacro:cuboid_inertia_def mass="1000" z="${altura_base}" x="1" y="1"/>
   </link>
   <link name="link1">
@@ -46,5 +60,5 @@
       <origin xyz="0 0 ${largo/2}" rpy="0 0 0" />
     </collision>
-    <xacro:default_inertial mass="${masa}" altoL="${largo}"/>
+    <xacro:default_inertial mass="${masa}" length="${largo}" radius="${ancho}"/>
   </link>
   <link name="link2">
@@ -62,5 +76,5 @@
       <origin xyz="0 0 ${largo/2}" rpy="0 0 0" />
     </collision>
-    <xacro:default_inertial mass="${masa}" altoL="${largo}"/>
+    <xacro:default_inertial mass="${masa}" length="${largo}" radius="${ancho}"/>
   </link>
   <link name="link3">
@@ -78,5 +92,5 @@
       <origin xyz="0 0 ${largo/2}" rpy="0 0 0" />
     </collision>
-    <xacro:default_inertial mass="${masa}" altoL="${largo}"/>
+    <xacro:default_inertial mass="${masa}" length="${largo}" radius="${ancho}"/>
   </link>
   <link name="link4">
@@ -94,5 +108,5 @@
       <origin xyz="0 0 ${largo/2}" rpy="0 0 0" />
     </collision>
-    <xacro:default_inertial mass="${masa}" altoL="${largo}"/>
+    <xacro:default_inertial mass="${masa}" length="${largo}" radius="${ancho}"/>
   </link>
   <link name="link5">
@@ -102,5 +116,5 @@
       </geometry>
       <origin xyz="0 0 ${ancho}" rpy="0 0 0" />
-      <material name="orange"/>
+      <material name="brown"/>
     </visual>
     <collision>
@@ -110,5 +124,5 @@
       <origin xyz="0 0 ${ancho}" rpy="0 0 0" />
     </collision>
-    <xacro:default_inertial mass="${masa/20}" altoL="${ancho}"/>
+    <xacro:default_inertial mass="${masa/20}" length="${ancho}" radius="${ancho}"/>
   </link>
   <joint name="joint0" type="fixed">

File: src/SimpleArm/urdf/materials.xacro (robot description, xacro)
@@ -17,5 +17,5 @@
   </material>
   <material name="brown">
-    <color rgba="${222/255} ${207/255} ${195/255} 1.0"/>
+    <color rgba="${222/255} ${207/255} ${195/255} 0.5"/>
   </material>
   <material name="red">

Commit message: Changed model effort limits

File: src/SimpleArm/urdf/SimpleArm.xacro (robot description, xacro)
@@ -7,4 +7,5 @@
   <xacro:property name="masa" value="5"/>
   <xacro:property name="delta" value="0.1"/>
+  <xacro:property name="pi" value="3.14"/>
   <xacro:macro name="cuboid_inertia_def" params="x y z mass">
     <inertial>
@@ -136,6 +137,7 @@
     <axis xyz="0 0 1"/>
     <dynamics damping="0.6"/>
-  </joint>
-  <joint name="joint2" type="continuous">
+     <limit effort="200" velocity="20" />
+  </joint>
+  <joint name="joint2" type="revolute">
     <parent link="link1"/>
     <child link="link2"/>
@@ -143,6 +145,7 @@
     <axis xyz="0 1 0"/>
     <dynamics damping="0.6"/>
-  </joint>
-  <joint name="joint3" type="continuous">
+    <limit effort="200" velocity="20" lower="${-pi/2}" upper="${pi/2}" />
+  </joint>
+  <joint name="joint3" type="revolute">
     <parent link="link2"/>
     <child link="link3"/>
@@ -150,6 +153,7 @@
     <axis xyz="0 1 0"/>
     <dynamics damping="0.6"/>
-  </joint>
-  <joint name="joint4" type="continuous">
+    <limit effort="90" velocity="20" lower="${-pi/2}" upper="${pi/2}" />
+  </joint>
+  <joint name="joint4" type="revolute">
     <parent link="link3"/>
     <child link="link4"/>
@@ -157,4 +161,5 @@
     <axis xyz="0 1 0"/>
     <dynamics damping="0.6"/>
+    <limit effort="40" velocity="20" lower="${-pi/2}" upper="${pi/2}" />
   </joint>
   <joint name="joint5" type="fixed">

Commit message: Moved sphere axis position to coincide with center

File: src/SimpleArm/urdf/SimpleArm.xacro (robot description, xacro)
@@ -116,5 +116,5 @@
         <sphere radius="${ancho}"/>
       </geometry>
-      <origin xyz="0 0 ${ancho}" rpy="0 0 0" />
+      <origin xyz="0 0 0" rpy="0 0 0" />
       <material name="brown"/>
     </visual>
@@ -123,5 +123,5 @@
         <sphere radius="${ancho}"/>
       </geometry>
-      <origin xyz="0 0 ${ancho}" rpy="0 0 0" />
+      <origin xyz="0 0 0" rpy="0 0 0" />
     </collision>
     <xacro:default_inertial mass="${masa/20}" length="${ancho}" radius="${ancho}"/>
@@ -166,5 +166,5 @@
     <parent link="link4"/>
     <child link="link5"/>
-    <origin xyz="0 0 ${largo}" rpy="0 0 0" />
+    <origin xyz="0 0 ${largo+ancho}" rpy="0 0 0" />
     </joint>
   <!-- Transmission -->

Commit message: a

File: src/SimpleArm/urdf/SimpleArm.xacro (robot description, xacro)
@@ -36,5 +36,5 @@
       <origin xyz="0 0 ${altura_base/2}" rpy="0 0 0"/>
       <geometry>
-        <box size="1 1 ${altura_base}"/>
+        <box size="0.2 0.2 ${altura_base}"/>
       </geometry>
     </visual>

Commit message: merge fix

File: src/SimpleArm/urdf/SimpleArm.xacro (robot description, xacro)
@@ -116,5 +116,5 @@
         <sphere radius="${ancho}"/>
       </geometry>
-      <origin xyz="0 0 0" rpy="0 0 0" />
+      <origin xyz="0 0 ${ancho}" rpy="0 0 0" />
       <material name="brown"/>
     </visual>
@@ -123,5 +123,5 @@
         <sphere radius="${ancho}"/>
       </geometry>
-      <origin xyz="0 0 0" rpy="0 0 0" />
+      <origin xyz="0 0 ${ancho}" rpy="0 0 0" />
     </collision>
     <xacro:default_inertial mass="${masa/20}" length="${ancho}" radius="${ancho}"/>
@@ -166,5 +166,5 @@
     <parent link="link4"/>
     <child link="link5"/>
-    <origin xyz="0 0 ${largo+ancho}" rpy="0 0 0" />
+    <origin xyz="0 0 ${largo}" rpy="0 0 0" />
     </joint>
   <!-- Transmission -->
